File: Hardware/foxmox.kicad_pcb (KiCad board)
At the start: 2 copper layers, 50 x 50 mm, 24 parts, among them P1 2.5mm plug, Q1 2N2222A, U1 PIC16F84, Y1 3.579MHz

Commit message: Final fixup before fab
Parts:
- moved C4 1.00 mm to (132.5, 63.5)
Routing:
- net Net-(C4-Pad2): track 39.4 -> 40.2 mm
- net Net-(U1-RB7): track 18.6 -> 19.2 mm

Commit message: Add open hardware and github silkscreens
Parts:
- added SYM1: Logo_Open_Hardware_Small, Symbol:OSHW-Logo2_7.3x6mm_SilkScreen, B.Cu at (135.0, 95.0)
Other:
- board text added: "https://github.com/k0swe/foxmox"
